Commit message: add mesh description

File: description/urdf/jaka_zu12.urdf (robot description, URDF)
Before this commit: robot jaka_zu12, 8 links, 7 joints
Links:
- link Link_0: geometry collision mesh filename=package://TetraPGA/description/meshes/jaka_zu12/base_link.S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; visual mesh filename=package://TetraPGA/description/meshes/jaka_zu12/base_link.S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
- link Link_1: geometry collision mesh filename=package://TetraPGA/description/meshes/jaka_zu12/1.STL; visual mesh filename=package://TetraPGA/description/meshes/jaka_zu12/1.STL
- link Link_2: geometry collision mesh filename=package://TetraPGA/description/meshes/jaka_zu12/2.STL; visual mesh filename=package://TetraPGA/description/meshes/jaka_zu12/2.STL
- link Link_3: geometry collision mesh filename=package://TetraPGA/description/meshes/jaka_zu12/3.STL; visual mesh filename=package://TetraPGA/description/meshes/jaka_zu12/3.STL
- link Link_4: geometry collision mesh filename=package://TetraPGA/description/meshes/jaka_zu12/4.STL; visual mesh filename=package://TetraPGA/description/meshes/jaka_zu12/4.STL
- link Link_5: geometry collision mesh filename=package://TetraPGA/description/meshes/jaka_zu12/5.STL; visual mesh filename=package://TetraPGA/description/meshes/jaka_zu12/5.STL
- link Link_6: geometry collision mesh filename=package://TetraPGA/description/meshes/jaka_zu12/6.STL; visual mesh filename=package://TetraPGA/description/meshes/jaka_zu12/6.STL
